File: dcdc_buck.kicad_sch (KiCad schematic)
At the start: 86 parts, among them IC1 CD4013BM96, J1 Conn_01x02_Socket, J2 Conn_01x02_Socket, J3 Conn_01x02_Socket, J4 Conn_01x02_Socket, Q1 IRF9540NPBF, Q11 MMBT3904, Q12 MMBT3906, Q13 MMBT3904, Q3 IRF9540NS, Q5 IRF9Z24N, Q6 MMBT3904, U1 TLV9151DBV, U2 TLV9151DBV, U3 TLV9151DBV, U4 TL431DBV, U6 INA241B4IDR

Commit message: made room for Version 1.1 (WiP)
Parts:
- removed C3: 10µF, Capacitor_SMD:C_0805_2012Metric, symbol Device:C
- removed C7: 1u, Capacitor_SMD:C_0402_1005Metric, symbol Device:C
- removed IC1: CD4013BM96, PZ:SOIC127P600X175-14N, symbol PZ:CD4013BM96
- removed Q1: IRF9540NPBF, Package_TO_SOT_THT:TO-220-3_Vertical, symbol Transistor_FET:IRF9540N
- removed Q3: IRF9540NS, Package_TO_SOT_SMD:TO-263-3_TabPin2, symbol Transistor_FET:IRF9540N
Other:
- note added: "Current-Sense"
- note added: "Einstellbare Referenz"
- note added: "Gate_Drive"
- note removed: "BJT level shifter + push-pull drive"
- note removed: "SMT"
- note removed: "bedrahtet"
- moved on the sheet: C12, C14, C15, C2, C4, C8, C9, CF2, D10, J2, J4, L1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
